File: effect.sch (KiCad schematic (older format))
At the start: 33 parts, among them Q1 2N7002, Q2 2N7002, U5 TL072, U6 TL072

Commit message: Added pot footprints
Parts:
- RV1, RV2, RV3, RV4, RV5, RV6: footprint (none) -> Potentiometer_THT:alpha_pot_16mm
Changed lines of the file:
@@
 F 0 "RV1" V 2085 5700 50  0000 C CNN
 F 1 "gain 1 (a500k)" V 1994 5700 50  0000 C CNN
-F 2 "" H 2200 5700 50  0001 C CNN
+F 2 "Potentiometer_THT:alpha_pot_16mm" H 2200 5700 50  0001 C CNN
 F 3 "~" H 2200 5700 50  0001 C CNN
 	1    2200 5700
@@
 F 0 "RV2" V 2085 6200 50  0000 C CNN
 F 1 "gain 2 (a500k)" V 1994 6200 50  0000 C CNN
-F 2 "" H 2200 6200 50  0001 C CNN
+F 2 "Potentiometer_THT:alpha_pot_16mm" H 2200 6200 50  0001 C CNN
 F 3 "~" H 2200 6200 50  0001 C CNN
 	1    2200 6200
@@
 F 0 "RV3" V 5300 6000 50  0000 R CNN
 F 1 "tone 1 (b100k)" V 5300 5800 50  0000 R CNN
-F 2 "" H 5450 5550 50  0001 C CNN
+F 2 "Potentiometer_THT:alpha_pot_16mm" H 5450 5550 50  0001 C CNN
 F 3 "~" H 5450 5550 50  0001 C CNN
 	1    5450 5550
@@
 F 0 "RV4" V 5300 6500 50  0000 R CNN
 F 1 "tone 2 (b100k)" V 5300 6300 50  0000 R CNN
-F 2 "" H 5450 6050 50  0001 C CNN
+F 2 "Potentiometer_THT:alpha_pot_16mm" H 5450 6050 50  0001 C CNN
 F 3 "~" H 5450 6050 50  0001 C CNN
 	1    5450 6050
@@
 F 0 "RV5" H 8931 5296 50  0000 R CNN
 F 1 "volume 1 (a100k)" H 8931 5205 50  0000 R CNN
-F 2 "" H 9000 5250 50  0001 C CNN
+F 2 "Potentiometer_THT:alpha_pot_16mm" H 9000 5250 50  0001 C CNN
 F 3 "~" H 9000 5250 50  0001 C CNN
 	1    9000 5250
@@
 F 0 "RV6" H 8931 6046 50  0000 R CNN
 F 1 "volume 2 (a100k)" H 8931 5955 50  0000 R CNN
-F 2 "" H 9000 6000 50  0001 C CNN
+F 2 "Potentiometer_THT:alpha_pot_16mm" H 9000 6000 50  0001 C CNN
 F 3 "~" H 9000 6000 50  0001 C CNN
 	1    9000 6000

Commit message: Use better schematic
Parts:
- removed Q1, Q2: 2N7002, Package_TO_SOT_SMD:SOT-23, symbol Transistor_FET:2N7002
- removed R4, R6: 10k, Resistor_SMD:R_0603_1608Metric, symbol Device:R
- removed unit 1 of U5
- removed unit 2 of U6
- added R?: 1M, Resistor_SMD:R_0603_1608Metric, symbol Device:R
- RV5: value volume 1 (a100k) -> volume 1 (a10k)
- RV6: value volume 2 (a100k) -> volume 2 (a10k)
Connections:
- net GND: no longer R5.2
- net Vref: now also R5.2, U6.3 (+), R?.1; no longer U6.2 (-)
- net gain_out: now also D5.1 (K)
- net tone_pin_2: now also U6.2 (-); no longer U6.3 (+)
- net at C7.1: now also U5.6 (-), R?.2
- net at C12.2, R12.1: now also C14.2
- net at D6.1 (K): now also D4.2 (A)
Other:
- moved on the sheet: C10, C11, C12, C13, C14, C7, C8, C9, D4, D5, D6, R10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

Commit message: wooooo
Parts:
- removed unit 3 of U6
- gave numbers to parts that had none: 1
- renumbered U6 to U5
Other:
- moved on the sheet: U5C
Changed lines of the file:
@@
 	8550 1650 8550 1750
 $Comp
-L Amplifier_Operational:TL072 U6
+L Amplifier_Operational:TL072 U5
 U 1 1 60C594E9
 P 6750 3750
-F 0 "U6" H 6750 4117 50  0000 C CNN
+F 0 "U5" H 6750 4117 50  0000 C CNN
 F 1 "TL072" H 6750 4026 50  0000 C CNN
 F 2 "Package_SO:SOIC-8_3.9x4.9mm_P1.27mm" H 6750 3750 50  0001 C CNN
@@
 L Amplifier_Operational:TL072 U5
 U 3 1 60C5E124
-P 6350 1550
-F 0 "U5" H 6308 1596 50  0000 L CNN
-F 1 "TL072" H 6308 1505 50  0000 L CNN
-F 2 "Package_SO:SOIC-8_3.9x4.9mm_P1.27mm" H 6350 1550 50  0001 C CNN
-F 3 "http://www.ti.com/lit/ds/symlink/tl071.pdf" H 6350 1550 50  0001 C CNN
-F 4 "C6961" H 6350 1550 50  0001 C CNN "LCSC"
-	3    6350 1550
+P 7950 1700
+F 0 "U5" H 7908 1746 50  0000 L CNN
+F 1 "TL072" H 7908 1655 50  0000 L CNN
+F 2 "Package_SO:SOIC-8_3.9x4.9mm_P1.27mm" H 7950 1700 50  0001 C CNN
+F 3 "http://www.ti.com/lit/ds/symlink/tl071.pdf" H 7950 1700 50  0001 C CNN
+F 4 "C6961" H 7950 1700 50  0001 C CNN "LCSC"
+	3    7950 1700
 	1    0    0    -1
 $EndComp
-$Comp
-L Amplifier_Operational:TL072 U6
-U 3 1 60C5FF70
-P 6850 1550
-F 0 "U6" H 6808 1596 50  0000 L CNN
-F 1 "TL072" H 6808 1505 50  0000 L CNN
-F 2 "Package_SO:SOIC-8_3.9x4.9mm_P1.27mm" H 6850 1550 50  0001 C CNN
-F 3 "http://www.ti.com/lit/ds/symlink/tl071.pdf" H 6850 1550 50  0001 C CNN
-F 4 "C6961" H 6850 1550 50  0001 C CNN "LCSC"
-	3    6850 1550
-	1    0    0    -1
-$EndComp
-Text GLabel 6250 1150 1    50   Input ~ 0
+Text GLabel 7850 1300 1    50   Input ~ 0
 9V
-Wire Wire Line
-	6250 1150 6250 1200
-Wire Wire Line
-	6250 1200 6750 1200
-Wire Wire Line
-	6750 1200 6750 1250
-Connection ~ 6250 1200
-Wire Wire Line
-	6250 1200 6250 1250
 $Comp
 L power:GND #PWR021
 U 1 1 60C68A88
-P 6250 1850
-F 0 "#PWR021" H 6250 1600 50  0001 C CNN
-F 1 "GND" H 6255 1677 50  0000 C CNN
-F 2 "" H 6250 1850 50  0001 C CNN
-F 3 "" H 6250 1850 50  0001 C CNN
-	1    6250 1850
-	1    0    0    -1
-$EndComp
-$Comp
-L power:GND #PWR022
-U 1 1 60C694DC
-P 6750 1850
-F 0 "#PWR022" H 6750 1600 50  0001 C CNN
-F 1 "GND" H 6755 1677 50  0000 C CNN
-F 2 "" H 6750 1850 50  0001 C CNN
-F 3 "" H 6750 1850 50  0001 C CNN
-	1    6750 1850
+P 7850 2000
+F 0 "#PWR021" H 7850 1750 50  0001 C CNN
+F 1 "GND" H 7855 1827 50  0000 C CNN
+F 2 "" H 7850 2000 50  0001 C CNN
+F 3 "" H 7850 2000 50  0001 C CNN
+	1    7850 2000
 	1    0    0    -1
 $EndComp
@@
 Vref
 $Comp
-L Device:R R?
+L Device:R R4
 U 1 1 615EDD61
 P 2200 3700
-F 0 "R?" H 2270 3746 50  0000 L CNN
+F 0 "R4" H 2270 3746 50  0000 L CNN
 F 1 "1M" H 2270 3655 50  0000 L CNN
 F 2 "Resistor_SMD:R_0603_1608Metric" V 2130 3700 50  0001 C CNN
@@
 Wire Wire Line
 	2200 3450 2200 3550
+Wire Wire Line
+	7850 1300 7850 1400
 $EndSCHEMATC
