File: template.kicad_pcb (KiCad board)
At the start: 2 copper layers, 95 x 65 mm, 54 parts, among them J1 power, J2 input, J3 output, J4 isp, K1 EC2-5NU, K2 EC2-5NU, K3 EC2-5NU, SW1 bypass switch, SW2 preset switch, U1 AMS1117-5.0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

Commit message: I think placement is done?
Parts:
- moved C2 32.6 mm to (132.1, 95.8), turned to 180 degrees
- moved R14 16.5 mm to (148.9, 101.3)
- moved C13 12.4 mm to (132.1, 101.0), turned to 180 degrees
- moved C5 12.2 mm to (159.1, 95.0)
- moved C8 9.06 mm to (139.9, 101.3), turned to 270 degrees
- moved U4 7.92 mm to (170.3, 84.6)
- moved R5 7.26 mm to (144.0, 101.3), turned to 90 degrees
- moved R1 6.68 mm to (153.7, 101.3)
- moved R4 6.12 mm to (144.0, 95.0), turned to 90 degrees
- moved C6 5.79 mm to (159.1, 101.3)
- moved R13 5.20 mm to (139.9, 95.0)
- moved R12 3.53 mm to (105.8, 101.3)
- moved R2 3.50 mm to (162.9, 101.3)
- moved C12 3.19 mm to (110.1, 101.3)
- moved C14 3.10 mm to (114.3, 101.3)
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
Commit message: so close
Parts:
- moved U3 7.64 mm to (113.8, 72.0)
- moved K1 4.72 mm to (111.4, 53.6)
- moved C4 1.66 mm to (153.5, 72.2)
- moved C3 1.39 mm to (150.8, 71.4)
- moved C1 0.99 mm to (148.4, 71.4)
- moved U4 0.77 mm to (171.1, 84.6)
- moved D1 0.30 mm to (151.1, 64.4)
- moved J1 0.30 mm to (131.0, 68.3)
- moved U1 0.28 mm to (151.1, 56.5)
- moved D2 0.28 mm to (97.5, 112.7)
- moved D3 0.28 mm to (167.5, 112.7)
- moved J4 0.19 mm to (134.8, 73.2)
Routing:
- net /effect/gain_out: track 0.00 -> 96.5 mm, vias 0 -> 4
- net /bypass_switch: track 0.00 -> 82.2 mm, vias 0 -> 4
- net 9V: track 0.00 -> 63.8 mm, vias 0 -> 2
- net Net-(D2-Pad2): track 0.00 -> 59.5 mm, vias 0 -> 1
- net /effect/tone_pin_3: track 0.00 -> 54.4 mm, vias 0 -> 3
- net /out: track 0.00 -> 47.0 mm
- net Net-(C8-Pad1): track 0.00 -> 43.7 mm, vias 0 -> 3
- net /preset_3_out_a: track 0.04 -> 40.7 mm
- net /miso: track 0.00 -> 37.2 mm, vias 0 -> 1
- net /effect/Vref: track 0.00 -> 34.1 mm, vias 0 -> 2
- net /preset_3_out_b: track 0.00 -> 32.8 mm
- net /effect/tone_pin_2: track 0.00 -> 29.5 mm, vias 0 -> 1
- net /return: track 0.00 -> 28.0 mm, vias 0 -> 1
- net /in: track 0.00 -> 26.2 mm
- net /bypass_led: track 0.00 -> 25.2 mm, vias 0 -> 3
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- added copper zone on B.Cu, net /5V
Other:
- board text added: "+"
- board text added: "-"

Commit message: So close
Routing:
- net /preset_relay: track 0.00 -> 60.2 mm, vias 0 -> 4
- net /send: track 4.10 -> 48.7 mm, vias 0 -> 2
- net /bypass_relay: track 0.00 -> 40.4 mm, vias 0 -> 2
- net /return: track 28.0 -> 53.7 mm, vias 1 -> 2
- net /preset_2_out_a: track 0.00 -> 20.5 mm, vias 0 -> 2
- net Net-(C11-Pad1): track 16.7 -> 36.3 mm
- net /out: track 47.0 -> 50.6 mm
- net /effect/tone_pin_3: track 54.4 -> 54.9 mm, vias 3 -> 4
- net /effect/tone_pin_2: vias 1 -> 2
Other:
- board text added: "overderive v1 beta"

Commit message: oh yeeaaa
Routing:
- net /miso: track 37.2 -> 62.7 mm, vias 1 -> 5
- net /bypass_led: track 25.2 -> 46.9 mm, vias 3 -> 7
- net /bypass_switch: track 82.2 -> 96.0 mm, vias 4 -> 6
- net /in: track 26.2 -> 27.2 mm, vias 0 -> 1
- net /return: vias 2 -> 4

Commit message: Sent it off 2 tha fab
Parts:
- removed G***: LOGO, dsp_dev_board:frankie
- added Ref**: Val**, text:logo, F.Cu at (95.9, 100.5)
Connections:
- U5 pad 5: Net-(C8-Pad1) -> Net-(C7-Pad1)
- U5 pad 6: Net-(C7-Pad1) -> Net-(C8-Pad1)
Routing:
- net Net-(C8-Pad1): track 43.7 -> 45.0 mm
- net Net-(C7-Pad1): track 10.8 -> 11.9 mm
Other:
- board text added: "JLCJLCJLCJLC"
- board text added: "a10k"
- board text added: "a500k"
- board text added: "b100k"
